Commit message: add functional motors

File: eolab_description/macros/core_sensors.xacro (robot description, xacro)
@@ -3,4 +3,7 @@
   <xacro:macro name="core_sensors" params="link">
     <gazebo>
+      <plugin filename="gz-sim-imu-system"
+        name="gz::sim::systems::Imu">
+      </plugin>
       <plugin filename="gz-sim-air-pressure-system"
         name="gz::sim::systems::AirPressure">
@@ -9,4 +12,8 @@
         name="gz::sim::systems::AirSpeed">
       </plugin>
+      <!-- This plugin is just for world -->
+      <!-- <plugin filename="gz-sim-apply-link-wrench-system" -->
+      <!--   name="gz::sim::systems::ApplyLinkWrench"> -->
+      <!-- </plugin> -->
       <plugin filename="gz-sim-navsat-system"
         name="gz::sim::systems::NavSat">
@@ -19,5 +26,5 @@
         <!-- TODO harley: check how good ogre2 is performing -->
         <!-- <render_engine>ogre2</render_engine> -->
-        <render_engine>ogre</render_engine>
+        <render_engine>ogre2</render_engine>
       </plugin>
       <!-- TODO harley: this looks like custom plugins, check if required -->
@@ -31,89 +38,84 @@
         <always_on>1</always_on>
         <update_rate>50</update_rate>
-        <air_pressure>
+        <!-- <air_pressure> -->
           <!-- Noise modeled after BMP390 -->
-          <pressure>
-            <noise type="gaussian">
-              <mean>0</mean>
-              <stddev>3</stddev>
-            </noise>
-          </pressure>
-        </air_pressure>
+        <!--   <pressure> -->
+        <!--     <noise type="gaussian"> -->
+        <!--       <mean>0</mean> -->
+        <!--       <stddev>3</stddev> -->
+        <!--     </noise> -->
+        <!--   </pressure> -->
+        <!-- </air_pressure> -->
       </sensor>
       <sensor name="magnetometer_sensor" type="magnetometer">
         <always_on>1</always_on>
         <update_rate>100</update_rate>
-        <magnetometer>
+        <!-- <magnetometer> -->
           <!-- TODO: update to fix units and coordinate system when we move past Harmonic -->
           <!-- See https://github.com/gazebosim/gz-sim/pull/2460 -->
           <!-- 3mgauss RMS: NOTE: noise is in tesla but sensor reports data in gauss -->
           <!-- Noise modeled after IIS2MDC -->
-          <x>
-            <noise type="gaussian">
-              <stddev>0.0001</stddev>
-            </noise>
-          </x>
-          <y>
-            <noise type="gaussian">
-              <stddev>0.0001</stddev>
-            </noise>
-          </y>
-          <z>
-            <noise type="gaussian">
-              <stddev>0.0001</stddev>
-            </noise>
-          </z>
-        </magnetometer>
+        <!--   <x> -->
+        <!--     <noise type="gaussian"> -->
+        <!--       <stddev>0.0001</stddev> -->
+        <!--     </noise> -->
+        <!--   </x> -->
+        <!--   <y> -->
+        <!--     <noise type="gaussian"> -->
+        <!--       <stddev>0.0001</stddev> -->
+        <!--     </noise> -->
+        <!--   </y> -->
+        <!--   <z> -->
+        <!--     <noise type="gaussian"> -->
+        <!--       <stddev>0.0001</stddev> -->
+        <!--     </noise> -->
+        <!--   </z> -->
+        <!-- </magnetometer> -->
       </sensor>
       <sensor name="imu_sensor" type="imu">
         <always_on>1</always_on>
         <update_rate>250</update_rate>
-        <imu>
-          <angular_velocity>
-            <!-- Noise modeled after IIM42653 -->
-            <!-- 0.05 deg/s converted to rad/s -->
-            <x>
-              <noise type="gaussian">
-                <mean>0.0</mean>
-                <stddev>0.0008726646</stddev>
-              </noise>
-            </x>
-            <y>
-              <noise type="gaussian">
-                <mean>0.0</mean>
-                <stddev>0.0008726646</stddev>
-              </noise>
-            </y>
-            <z>
-              <noise type="gaussian">
-                <mean>0.0</mean>
-                <stddev>0.0008726646</stddev>
-              </noise>
-            </z>
-          </angular_velocity>
-          <linear_acceleration>
-            <!-- Noise modeled after IIM42653 -->
-            <!-- X & Y axis: 0.65 mg-rms converted to m/ss -->
-            <x>
-              <noise type="gaussian">
-                <mean>0.0</mean>
-                <stddev>0.00637</stddev>
-              </noise>
-            </x>
-            <y>
-              <noise type="gaussian">
-                <mean>0.0</mean>
-                <stddev>0.00637</stddev>
-              </noise>
-            </y>
-            <!-- Z axis: 0.70 mg-rms converted to m/ss-->
-            <z>
-              <noise type="gaussian">
-                <mean>0.0</mean>
-                <stddev>0.00686</stddev>
-              </noise>
-            </z>
-          </linear_acceleration>
-        </imu>
+        <!-- <imu> -->
+        <!--   <angular_velocity> -->
+        <!--     <x> -->
+        <!--       <noise type="gaussian"> -->
+        <!--         <mean>0.0</mean> -->
+        <!--         <stddev>0.0008726646</stddev> -->
+        <!--       </noise> -->
+        <!--     </x> -->
+        <!--     <y> -->
+        <!--       <noise type="gaussian"> -->
+        <!--         <mean>0.0</mean> -->
+        <!--         <stddev>0.0008726646</stddev> -->
+        <!--       </noise> -->
+        <!--     </y> -->
+        <!--     <z> -->
+        <!--       <noise type="gaussian"> -->
+        <!--         <mean>0.0</mean> -->
+        <!--         <stddev>0.0008726646</stddev> -->
+        <!--       </noise> -->
+        <!--     </z> -->
+        <!--   </angular_velocity> -->
+        <!--   <linear_acceleration> -->
+        <!--     <x> -->
+        <!--       <noise type="gaussian"> -->
+        <!--         <mean>0.0</mean> -->
+        <!--         <stddev>0.00637</stddev> -->
+        <!--       </noise> -->
+        <!--     </x> -->
+        <!--     <y> -->
+        <!--       <noise type="gaussian"> -->
+        <!--         <mean>0.0</mean> -->
+        <!--         <stddev>0.00637</stddev> -->
+        <!--       </noise> -->
+        <!--     </y> -->
+        <!--     <z> -->
+        <!--       <noise type="gaussian"> -->
+        <!--         <mean>0.0</mean> -->
+        <!--         <stddev>0.00686</stddev> -->
+        <!--       </noise> -->
+        <!--     </z> -->
+        <!--   </linear_acceleration> -->
+        <!-- </imu> -->
       </sensor>
       <sensor name="navsat_sensor" type="navsat">

File: eolab_description/xacros/phoenix.urdf.xacro (robot description, xacro)
@@ -2,5 +2,4 @@
   <xacro:property name="root_frame" value="base_link"/>
   <xacro:include filename="$(find eolab_description)/macros/core_sensors.xacro"/>
-  <xacro:core_sensors link="${root_frame}"/>
   <xacro:macro name="box_inertia" params="m w h d">
     <inertial>
@@ -10,6 +9,4 @@
     </inertial>
   </xacro:macro>
-  <!-- TODOs: -->
-  <!-- add inertial and mass -->
   <link name="${root_frame}">
     <visual>
@@ -25,11 +22,61 @@
     <xacro:box_inertia m="2" w="0.3" h="0.3" d="0.3"/>
   </link>
-    <link name="base_footprint">
-      <xacro:box_inertia m="0.5" w="0.01" d="0.01" h="0.01"/>
+  <xacro:core_sensors link="${root_frame}"/>
+  <xacro:macro name="phoenix_rotor" params="number parent direction *origin">
+    <link name="rotor_${number}">
+      <visual>
+        <geometry>
+          <box size="0.4 0.04 0.01"/>
+        </geometry>
+      </visual>
+      <collision>
+        <geometry>
+          <box size="0.4 0.04 0.01"/>
+        </geometry>
+      </collision>
+      <xacro:box_inertia m="0.1" w="0.4" h="0.04" d="0.01"/>
     </link>
-    <joint name="base_joint" type="fixed">
-      <parent link="${root_frame}" />
-      <child link="base_footprint" />
-      <origin xyz="0 0 0" rpy="0 0 0" />
+    <joint name="rotor_${number}_joint" type="continuous">
+      <parent link="${parent}"/>
+      <child link="rotor_${number}"/>
+      <xacro:insert_block name="origin" />
+      <axis xyz="0 0 1"/>
     </joint>
+    <gazebo>
+      <plugin filename="gz-sim-multicopter-motor-model-system" name="gz::sim::systems::MulticopterMotorModel">
+        <jointName>rotor_${number}_joint</jointName>
+        <linkName>rotor_${number}</linkName>
+        <turningDirection>${direction}</turningDirection>
+        <timeConstantUp>0.0125</timeConstantUp>
+        <timeConstantDown>0.025</timeConstantDown>
+        <maxRotVelocity>1000.0</maxRotVelocity>
+        <motorConstant>8.54858e-06</motorConstant>
+        <momentConstant>0.016</momentConstant>
+        <commandSubTopic>command/motor_speed</commandSubTopic>
+        <motorNumber>${number}</motorNumber>
+        <rotorDragCoefficient>8.06428e-05</rotorDragCoefficient>
+        <rollingMomentCoefficient>1e-06</rollingMomentCoefficient>
+        <rotorVelocitySlowdownSim>10</rotorVelocitySlowdownSim>
+        <motorType>velocity</motorType>
+      </plugin>
+    </gazebo>
+  </xacro:macro>
+  <xacro:phoenix_rotor number="0" parent="${root_frame}" direction="cw">
+    <origin xyz="0.58 0 0.4" rpy="0 0 0"/>
+  </xacro:phoenix_rotor>
+  <xacro:phoenix_rotor number="1" parent="${root_frame}" direction="ccw">
+    <origin xyz="-0.58 0 0.4" rpy="0 0 0"/>
+  </xacro:phoenix_rotor>
+  <xacro:phoenix_rotor number="2" parent="${root_frame}" direction="cw">
+    <origin xyz="-0.29 -0.51 0.4" rpy="0 0 0"/>
+  </xacro:phoenix_rotor>
+  <xacro:phoenix_rotor number="3" parent="${root_frame}" direction="ccw">
+    <origin xyz="0.29 0.51 0.4" rpy="0 0 0"/>
+  </xacro:phoenix_rotor>
+  <xacro:phoenix_rotor number="4" parent="${root_frame}" direction="ccw">
+    <origin xyz="0.29 -0.51 0.4" rpy="0 0 0"/>
+  </xacro:phoenix_rotor>
+  <xacro:phoenix_rotor number="5" parent="${root_frame}" direction="cw">
+    <origin xyz="-0.29 0.51 0.4" rpy="0 0 0"/>
+  </xacro:phoenix_rotor>
 </robot>
