Commit message: fix motor physics and number (takeoff)

File: eolab_description/drones/phoenix.urdf.xacro (robot description, xacro)
@@ -5,5 +5,5 @@
   <xacro:macro name="box_inertia" params="m w h d">
     <inertial>
-      <origin xyz="0 0 0" rpy="${pi/2} 0 ${pi/2}"/>
+      <origin xyz="0 0 0" rpy="0 0 0"/>
       <mass value="${m}"/>
       <inertia ixx="${(m/12) * (h*h + d*d)}" ixy="0.0" ixz="0.0" iyy="${(m/12) * (w*w + d*d)}" iyz="0.0" izz="${(m/12) * (w*w + h*h)}"/>
@@ -21,29 +21,28 @@
       </geometry>
     </collision>
-    <!-- <xacro:box_inertia m="2" w="0.3" h="0.3" d="0.3"/> -->
     <inertial>
       <origin xyz="0 0 0" rpy="0 0 0"/>
       <mass value="5.5"/>
-      <inertia ixx="0.02" ixy="0" ixz="0" iyy="0.021" iyz="0.0" izz="0.04"/>
+      <inertia ixx="0.4613" ixy="0" ixz="0" iyy="0.6115" iyz="0.0" izz="1.0669"/>
     </inertial>
   </link>
   <xacro:core_sensors link="${root_frame}"/>
   <xacro:t_motor_mf2009 number="0" parent="${root_frame}" direction="cw">
-    <origin xyz="0.58 0 0.05" rpy="0 0 0"/>
+    <origin xyz="0 -0.58 0.05" rpy="0 0 0"/>
   </xacro:t_motor_mf2009>
   <xacro:t_motor_mf2009 number="1" parent="${root_frame}" direction="ccw">
-    <origin xyz="-0.58 0 0.05" rpy="0 0 0"/>
+    <origin xyz="0 0.58 0.05" rpy="0 0 0"/>
   </xacro:t_motor_mf2009>
   <xacro:t_motor_mf2009 number="2" parent="${root_frame}" direction="cw">
-    <origin xyz="-0.29 -0.51 0.05" rpy="0 0 0"/>
+    <origin xyz="0.51 0.29 0.05" rpy="0 0 0"/>
   </xacro:t_motor_mf2009>
   <xacro:t_motor_mf2009 number="3" parent="${root_frame}" direction="ccw">
-    <origin xyz="0.29 0.51 0.05" rpy="0 0 0"/>
+    <origin xyz="-0.51 -0.29 0.05" rpy="0 0 0"/>
   </xacro:t_motor_mf2009>
   <xacro:t_motor_mf2009 number="4" parent="${root_frame}" direction="ccw">
-    <origin xyz="0.29 -0.51 0.05" rpy="0 0 0"/>
+    <origin xyz="0.51 -0.29 0.05" rpy="0 0 0"/>
   </xacro:t_motor_mf2009>
   <xacro:t_motor_mf2009 number="5" parent="${root_frame}" direction="cw">
-    <origin xyz="-0.29 0.51 0.05" rpy="0 0 0"/>
+    <origin xyz="-0.51 0.29 0.05" rpy="0 0 0"/>
   </xacro:t_motor_mf2009>
 </robot>

File: eolab_description/props/t_motor_mf2009.xacro (robot description, xacro)
@@ -6,7 +6,8 @@
     <xacro:property name="prop_weight" value="0.059"/>
     <!-- Recommended Thrust/RPM: 3.5kg / 4700RPM -->
-    <!-- Recommended Max Thrust/RPM: 9kg / 7000RPM-->
-    <xacro:property name="prop_max_rpm" value="7000"/>
+    <!-- Recommended Max Thrust/RPM: 9kg / 7000RPM 733 rad/s -->
+    <xacro:property name="prop_max_rad_per_sec" value="733"/>
     <link name="rotor_${number}">
+      <origin xyz="0 0 0" rpy="0 0 0"/>
       <visual>
         <geometry>
@@ -19,4 +20,7 @@
         </geometry>
       </collision>
+      <mass value="${prop_weight}"/>
+      <!-- real value heavy-->
+      <!-- <mass value="5.5"/> -->
       <xacro:box_inertia m="${prop_weight}" w="${prop_diameter}" h="0.04" d="0.01"/>
     </link>
@@ -34,9 +38,9 @@
         <timeConstantUp>0.0125</timeConstantUp>
         <timeConstantDown>0.025</timeConstantDown>
-        <maxRotVelocity>${prop_max_rpm}</maxRotVelocity>
-        <motorConstant>8.54858e-06</motorConstant>
+        <maxRotVelocity>${prop_max_rad_per_sec}</maxRotVelocity>
+        <motorConstant>1.6378e-04</motorConstant> <!-- compute from: T/rad sec)2 -->
         <momentConstant>0.016</momentConstant>
         <commandSubTopic>command/motor_speed</commandSubTopic>
-        <motorNumber>${number}</motorNumber>
+        <actuator_number>${number}</actuator_number>
         <rotorDragCoefficient>8.06428e-05</rotorDragCoefficient>
         <rollingMomentCoefficient>1e-06</rollingMomentCoefficient>

Commit message: fix drone orientation yaw

File: eolab_description/drones/phoenix.urdf.xacro (robot description, xacro)
@@ -12,4 +12,5 @@
   <link name="${root_frame}">
     <visual>
+      <origin xyz="0 0 0" rpy="0 0 ${pi/2}"/>
       <geometry>
         <mesh filename="file://$(find eolab_description)/drones/meshes/phoenix.obj" scale="1 1 1"/>
@@ -17,4 +18,5 @@
     </visual>
     <collision>
+      <origin xyz="0 0 0" rpy="0 0 ${pi/2}"/>
       <geometry>
         <mesh filename="file://$(find eolab_description)/drones/meshes/phoenix.obj" scale="1 1 1"/>
@@ -22,5 +24,6 @@
     </collision>
     <inertial>
-      <origin xyz="0 0 0" rpy="0 0 0"/>
+      <origin xyz="0 0 0" rpy="0 0 ${pi/2}"/>
+      <!-- TODO harley: add battery weight -->
       <mass value="5.5"/>
       <inertia ixx="0.4613" ixy="0" ixz="0" iyy="0.6115" iyz="0.0" izz="1.0669"/>

Commit message: fix mass of base to include battery

File: eolab_description/drones/phoenix.urdf.xacro (robot description, xacro)
@@ -26,5 +26,5 @@
       <origin xyz="0 0 0" rpy="0 0 ${pi/2}"/>
       <!-- TODO harley: add battery weight -->
-      <mass value="5.5"/>
+      <mass value="6.5"/>
       <inertia ixx="0.4613" ixy="0" ixz="0" iyy="0.6115" iyz="0.0" izz="1.0669"/>
     </inertial>

Commit message: rename folder

File: eolab_description/drones/phoenix.urdf.xacro (robot description, xacro)
@@ -2,5 +2,5 @@
   <xacro:property name="root_frame" value="base_link"/>
   <xacro:include filename="$(find eolab_description)/payloads/core_sensors.xacro"/>
-  <xacro:include filename="$(find eolab_description)/props/t_motor_mf2009.xacro"/>
+  <xacro:include filename="$(find eolab_description)/propulsions/t_motor_mf2009.xacro"/>
   <xacro:macro name="box_inertia" params="m w h d">
     <inertial>

File: eolab_description/drones/protoflyer.urdf.xacro (robot description, xacro)
@@ -2,5 +2,6 @@
   <xacro:property name="root_frame" value="base_link"/>
   <xacro:include filename="$(find eolab_description)/payloads/core_sensors.xacro"/>
-  <xacro:include filename="$(find eolab_description)/props/dji_e305.xacro"/>
+  <xacro:include filename="$(find eolab_description)/payloads/rgb_generic.xacro"/>
+  <xacro:include filename="$(find eolab_description)/propulsions/dji_e305.xacro"/>
   <xacro:macro name="box_inertia" params="m w h d">
     <inertial>
@@ -32,4 +33,11 @@
   </link>
   <xacro:core_sensors link="${root_frame}"/>
+  <xacro:rgb_generic
+   name="rgb_camera"
+   parent_link="${root_frame}"
+   namespace=""
+   system="">
+    <origin xyz="0 0 -0.05" rpy="0 0 0"/>
+  </xacro:rgb_generic>
   <xacro:dji_e305 number="0" parent="${root_frame}" direction="ccw">
     <origin xyz="0.158 -0.158 0.05" rpy="0 0 0"/>
