Commit message: add protolfyer params

File: eolab_description/drones/protoflyer.urdf.xacro (robot description, xacro)
@@ -26,5 +26,5 @@
       <!-- <origin xyz="0 0 0" rpy="0 0 ${pi/2}"/> -->
       <!-- TODO harley: add battery weight -->
-      <mass value="1.5"/>
+      <mass value="0.5"/>
       <!-- <inertia ixx="1.552e7" ixy="0.003" ixz="0" iyy="1.549e7" iyz="0.003" izz="3.068e7"/> -->
       <inertia ixx="1.552e7" ixy="0.003" ixz="0" iyy="1.549e7" iyz="0.003" izz="3.068e7"/>

Commit message: change camera view to look downward

File: eolab_description/drones/protoflyer.urdf.xacro (robot description, xacro)
@@ -38,5 +38,5 @@
    namespace=""
    system="gz">
-    <origin xyz="0 0 -0.05" rpy="0 0 0"/>
+    <origin xyz="0 0 -0.05" rpy="0 ${radians(90)} 0"/>
   </xacro:rgb_generic>
   <xacro:dji_e305 number="0" parent="${root_frame}" direction="ccw">

Commit message: fix collision box

File: eolab_description/drones/protoflyer.urdf.xacro (robot description, xacro)
@@ -21,5 +21,5 @@
       <!-- <origin xyz="0 0 0" rpy="0 0 ${pi/2}"/> -->
       <geometry>
-        <box size="0.39 0.39 0.25"/>
+        <box size="0.39 0.39 0.39"/>
       </geometry>
     </collision>

Commit message: fix inertial matrix

File: eolab_description/drones/protoflyer.urdf.xacro (robot description, xacro)
@@ -4,14 +4,17 @@
   <xacro:include filename="$(find eolab_description)/payloads/rgb_generic.xacro"/>
   <xacro:include filename="$(find eolab_description)/propulsions/dji_e305.xacro"/>
-  <xacro:macro name="box_inertia" params="m w h d">
+  <xacro:macro name="box_inertial" params="mass x y z xyz:='0 0 0' rpy:='0 0 0'">
     <inertial>
-      <origin xyz="0 0 0" rpy="0 0 0"/>
-      <mass value="${m}"/>
-      <inertia ixx="${(m/12) * (h*h + d*d)}" ixy="0.0" ixz="0.0" iyy="${(m/12) * (w*w + d*d)}" iyz="0.0" izz="${(m/12) * (w*w + h*h)}"/>
+      <origin xyz="${xyz}" rpy="${rpy}"/>
+      <mass value="${mass}"/>
+      <inertia
+        ixx="${(1/12.0)*mass*(y*y + z*z)}"
+        iyy="${(1/12.0)*mass*(x*x + z*z)}"
+        izz="${(1/12.0)*mass*(x*x + y*y)}"
+        ixy="0.0" ixz="0.0" iyz="0.0"/>
     </inertial>
   </xacro:macro>
   <link name="${root_frame}">
     <visual>
-      <!-- <origin xyz="0 0 0" rpy="0 0 ${pi/2}"/> -->
       <geometry>
         <mesh filename="file://$(find eolab_description)/drones/meshes/protoflyer.obj" scale="1 1 1"/>
@@ -19,16 +22,9 @@
     </visual>
     <collision>
-      <!-- <origin xyz="0 0 0" rpy="0 0 ${pi/2}"/> -->
       <geometry>
         <box size="0.39 0.39 0.39"/>
       </geometry>
     </collision>
-    <inertial>
-      <!-- <origin xyz="0 0 0" rpy="0 0 ${pi/2}"/> -->
-      <!-- TODO harley: add battery weight -->
-      <mass value="0.5"/>
-      <!-- <inertia ixx="1.552e7" ixy="0.003" ixz="0" iyy="1.549e7" iyz="0.003" izz="3.068e7"/> -->
-      <inertia ixx="1.552e7" ixy="0.003" ixz="0" iyy="1.549e7" iyz="0.003" izz="3.068e7"/>
-    </inertial>
+    <xacro:box_inertial mass="0.5" x="0.4" y="0.4" z="0.4"/>
   </link>
   <xacro:core_sensors link="${root_frame}"/>

File: eolab_description/propulsions/dji_e305.xacro (robot description, xacro)
@@ -18,8 +18,6 @@
         </geometry>
       </collision>
-      <mass value="${prop_weight}"/>
       <!-- real value heavy-->
-      <!-- <mass value="5.5"/> -->
-      <xacro:box_inertia m="${prop_weight}" w="${prop_diameter}" h="0.04" d="0.01"/>
+      <xacro:box_inertial mass="${prop_weight}" x="${prop_diameter}" y="0.04" z="0.01"/>
     </link>
     <joint name="rotor_${number}_joint" type="continuous">

Commit message: refactor launch system

File: eolab_description/drones/protoflyer.urdf.xacro (robot description, xacro)
@@ -1,7 +1,9 @@
 <robot name="protoflyer" xmlns:xacro="http://www.ros.org/wiki/xacro">
-  <xacro:property name="root_frame" value="base_link"/>
   <xacro:include filename="$(find eolab_description)/payloads/core_sensors.xacro"/>
   <xacro:include filename="$(find eolab_description)/payloads/rgb_generic.xacro"/>
   <xacro:include filename="$(find eolab_description)/propulsions/dji_e305.xacro"/>
+  <!-- <xacro:arg name="drone_name" default="protoflyer"/> -->
+  <!-- <xacro:property name="root_frame" value="$(arg drone_name)_base_link"/> -->
+  <xacro:property name="root_frame" value="base_link"/>
   <xacro:macro name="box_inertial" params="mass x y z xyz:='0 0 0' rpy:='0 0 0'">
     <inertial>
@@ -29,10 +31,7 @@
   </link>
   <xacro:core_sensors link="${root_frame}"/>
-  <xacro:rgb_generic
-   name="rgb_camera"
-   parent_link="${root_frame}"
-   namespace=""
-   system="gz">
+  <xacro:rgb_generic name="rgb_camera" parent_link="${root_frame}" system="gz">
     <origin xyz="0 0 -0.05" rpy="0 ${radians(90)} 0"/>
+      <!-- rotation in roll to look downward -->
   </xacro:rgb_generic>
   <xacro:dji_e305 number="0" parent="${root_frame}" direction="ccw">

File: eolab_description/payloads/core_sensors.xacro (robot description, xacro)
@@ -2,33 +2,13 @@
   <!-- link: name of the link to attach all the sensors -->
   <xacro:macro name="core_sensors" params="link">
-    <gazebo>
-      <plugin filename="gz-sim-imu-system"
-        name="gz::sim::systems::Imu">
-      </plugin>
-      <plugin filename="gz-sim-air-pressure-system"
-        name="gz::sim::systems::AirPressure">
-      </plugin>
-      <plugin filename="gz-sim-air-speed-system"
-        name="gz::sim::systems::AirSpeed">
-      </plugin>
-      <!-- This plugin is just for world -->
-      <!-- <plugin filename="gz-sim-apply-link-wrench-system" -->
-      <!--   name="gz::sim::systems::ApplyLinkWrench"> -->
-      <!-- </plugin> -->
-      <plugin filename="gz-sim-navsat-system"
-        name="gz::sim::systems::NavSat">
-      </plugin>
-      <plugin filename="gz-sim-magnetometer-system"
-        name="gz::sim::systems::Magnetometer">
-      </plugin>
-      <plugin filename="gz-sim-sensors-system"
-        name="gz::sim::systems::Sensors">
-        <!-- TODO harley: check how good ogre2 is performing -->
-        <!-- <render_engine>ogre2</render_engine> -->
-        <render_engine>ogre2</render_engine>
-      </plugin>
-    </gazebo>
-    <!-- ALL sensors are attach to the "link" property -->
-    <!-- this reference is important to go from XACRO->URDF->SDF -->
+    <!-- All sensors used here are initialized at the world level. -->
+    <!-- Instead of adding them to each world, we use -->
+    <!-- eolab_description/gz-configs/server.config -->
+    <!-- to attach them to any world that uses our server.config. -->
+    <!-- All sensors are attached to the "link" property. -->
+    <!-- This reference is important for the conversion chain: XACRO -> URDF -> SDF. -->
+    <!-- IMPORTANT: DO NOT change the sensor names. -->
+    <!-- For example, PX4 looks for names like "air_pressure_sensor" -->
+    <!-- specifically to bridge gz-sensors to PX4. -->
     <gazebo reference="${link}">
       <sensor name="air_pressure_sensor" type="air_pressure">

Commit message: refactor launch system and rest of components

File: eolab_description/drones/protoflyer.urdf.xacro (robot description, xacro)
@@ -17,5 +17,11 @@
     </inertial>
   </xacro:macro>
-  <link name="${root_frame}">
+  <link name="${root_frame}"/>
+  <joint name="body_frame_joint" type="fixed">
+    <origin xyz="0 0 0" rpy="0 0 0"/>
+    <parent link="${root_frame}"/>
+    <child link="body_frame_link"/>
+  </joint>
+  <link name="body_frame_link">
     <visual>
       <geometry>

Commit message: fix tf links

File: eolab_description/drones/protoflyer.urdf.xacro (robot description, xacro)
@@ -5,5 +5,5 @@
   <!-- <xacro:arg name="drone_name" default="protoflyer"/> -->
   <!-- <xacro:property name="root_frame" value="$(arg drone_name)_base_link"/> -->
-  <xacro:property name="root_frame" value="base_link"/>
+  <xacro:property name="root_frame" value="body_frame"/>
   <xacro:macro name="box_inertial" params="mass x y z xyz:='0 0 0' rpy:='0 0 0'">
     <inertial>
@@ -17,11 +17,11 @@
     </inertial>
   </xacro:macro>
-  <link name="${root_frame}"/>
-  <joint name="body_frame_joint" type="fixed">
+  <link name="base_link"/>
+  <joint name="${root_frame}_joint" type="fixed">
     <origin xyz="0 0 0" rpy="0 0 0"/>
-    <parent link="${root_frame}"/>
-    <child link="body_frame_link"/>
+    <parent link="base_link"/>
+    <child link="${root_frame}_link"/>
   </joint>
-  <link name="body_frame_link">
+  <link name="${root_frame}_link">
     <visual>
       <geometry>
@@ -36,5 +36,5 @@
     <xacro:box_inertial mass="0.5" x="0.4" y="0.4" z="0.4"/>
   </link>
-  <xacro:core_sensors link="${root_frame}"/>
+  <xacro:core_sensors link="${root_frame}_link"/>
   <xacro:rgb_generic name="rgb_camera" parent_link="${root_frame}" system="gz">
     <origin xyz="0 0 -0.05" rpy="0 ${radians(90)} 0"/>
